File: tiny328.kicad_pcb (KiCad board)
At the start: 2 copper layers, 35.1 x 22.4 mm, 20 parts, among them IC1 ATMEGA328P-A, U1 RFM12, U2 MCP1702, Y1 16MHz

Commit message: more routing, mounting holes
Parts:
- added 1PIN: P***, 1pin, F.Cu at (37.2, 25.1)
- added 1PIN: P***, 1pin, F.Cu at (61.2, 25.1)
- added JP9: PWR2, SIL-2A, F.Cu at (63.0, 31.5)
- JP7: value PWR IN -> PWR1; footprint SIL-3A -> SIL-2A
- U2: value MCP1702 -> MCP1702T-3302E/CB
- moved C1 10.3 mm to (43.9, 30.0), turned to 135 degrees
- moved JP7 8.89 mm to (63.0, 18.8)
- moved JP8 2.54 mm to (60.5, 17.5)
- moved Y1 2.54 mm to (39.1, 31.0)
- moved C3 2.17 mm to (60.5, 20.4)
- moved C5 2.04 mm to (32.5, 22.2)
- moved C6 2.04 mm to (32.5, 20.2)
- moved R1 1.76 mm to (41.9, 20.7)
- moved U2 1.47 mm to (33.1, 25.2)
- moved C4 1.27 mm to (41.4, 24.4)
- moved C7 1.17 mm to (33.4, 28.2)
- moved JP5 0.77 mm to (39.6, 27.1), turned to 90 degrees
Routing:
- net GND: track 52.8 -> 90.1 mm, vias 5 -> 2
- net 3V3: track 74.9 -> 64.3 mm
- net +5V: track 52.6 -> 60.7 mm, vias 3 -> 2
- net /D3: track 14.5 -> 18.8 mm
- net /D4: track 16.7 -> 20.3 mm
- net N-0000013: track 6.05 -> 9.54 mm
- net N-0000037: track 18.7 -> 22.1 mm
- net /A7: track 14.9 -> 11.5 mm
- net /A0: track 45.6 -> 42.2 mm
- net N-0000012: track 6.59 -> 9.13 mm
- net /D2: track 19.3 -> 21.2 mm
- net /D12/MISO: track 37.3 -> 35.5 mm
- net /D1/TX: track 34.4 -> 32.8 mm
- net /D0/RX: track 33.8 -> 33.1 mm
- net N-000009: track 3.36 -> 4.01 mm
