File: tiny328.sch (KiCad schematic (older format))
At the start: 20 parts, among them IC1 ATMEGA328P-A, U1 RFM12, U2 MCP1702T-3302E/CB, Y1 16MHz

Commit message: more routing, mounting holes
Parts:
- added JP9: PWR2, ~, symbol CONN_2
- JP7: value PWR IN -> PWR1; symbol CONN_3 -> CONN_2
Connections:
- wire segments 42 -> 45
Changed lines of the file:
@@
 Sheet 1 1
 Title ""
-Date "28 sep 2014"
+Date "3 oct 2014"
 Rev ""
 Comp ""
@@
 $EndComp
 $Comp
-L CONN_3 JP7
+L CONN_2 JP7
 U 1 1 542580DE
 P 5650 2650
 F 0 "JP7" V 5600 2650 50  0000 C CNN
-F 1 "PWR IN" V 5700 2650 40  0000 C CNN
+F 1 "PWR1" V 5700 2650 40  0000 C CNN
 F 2 "~" H 5650 2650 60  0000 C CNN
 F 3 "~" H 5650 2650 60  0000 C CNN
@@
 Wire Wire Line
 	5000 2650 5300 2650
-Text Label 5300 2750 2    60   ~ 0
+Text Label 5300 2950 2    60   ~ 0
 3V3
 Text Label 7400 1500 2    60   ~ 0
@@
 Text Label 4350 3000 0    60   ~ 0
 RESET
+$Comp
+L CONN_2 JP9
+U 1 1 542EF452
+P 5650 3050
+F 0 "JP9" V 5600 3050 40  0000 C CNN
+F 1 "PWR2" V 5700 3050 40  0000 C CNN
+F 2 "~" H 5650 3050 60  0000 C CNN
+F 3 "~" H 5650 3050 60  0000 C CNN
+	1    5650 3050
+	1    0    0    -1
+$EndComp
+Wire Wire Line
+	5300 2650 5300 2750
+Wire Wire Line
+	5300 3150 5050 3150
+Wire Wire Line
+	5050 3150 5050 2650
+Connection ~ 5050 2650
 $EndSCHEMATC

Commit message: all connected, flooded
Parts:
- added R2, R3: 100K, ~, symbol R
Connections:
- wire segments 45 -> 49
Other:
- moved on the sheet: R1
Changed lines of the file:
@@
 Sheet 1 1
 Title ""
-Date "3 oct 2014"
+Date "27 oct 2014"
 Rev ""
 Comp ""
@@
 NoConn ~ 5300 1950
 $Comp
-L GND #PWR01
+L GND #PWR10
 U 1 1 5425AD89
 P 5300 2050
-F 0 "#PWR01" H 5300 2050 30  0001 C CNN
+F 0 "#PWR10" H 5300 2050 30  0001 C CNN
 F 1 "GND" H 5300 1980 30  0001 C CNN
 F 2 "" H 5300 2050 60  0000 C CNN
@@
 5V
 $Comp
-L GND #PWR02
+L GND #PWR9
 U 1 1 5425ADEE
 P 5000 2850
-F 0 "#PWR02" H 5000 2850 30  0001 C CNN
+F 0 "#PWR9" H 5000 2850 30  0001 C CNN
 F 1 "GND" H 5000 2780 30  0001 C CNN
 F 2 "" H 5000 2850 60  0000 C CNN
@@
 5V
 $Comp
-L GND #PWR03
+L GND #PWR13
 U 1 1 5426FA0B
 P 6950 5000
-F 0 "#PWR03" H 6950 5000 30  0001 C CNN
+F 0 "#PWR13" H 6950 5000 30  0001 C CNN
 F 1 "GND" H 6950 4930 30  0001 C CNN
 F 2 "" H 6950 5000 60  0000 C CNN
@@
 	6350 4900 6300 4900
 $Comp
-L GND #PWR04
+L GND #PWR11
 U 1 1 5426FB80
 P 5350 5250
-F 0 "#PWR04" H 5350 5250 30  0001 C CNN
+F 0 "#PWR11" H 5350 5250 30  0001 C CNN
 F 1 "GND" H 5350 5180 30  0001 C CNN
 F 2 "" H 5350 5250 60  0000 C CNN
@@
 $EndComp
 $Comp
-L GND #PWR05
+L GND #PWR12
 U 1 1 5426FBC0
 P 6000 4100
-F 0 "#PWR05" H 6000 4100 30  0001 C CNN
+F 0 "#PWR12" H 6000 4100 30  0001 C CNN
 F 1 "GND" H 6000 4030 30  0001 C CNN
 F 2 "" H 6000 4100 60  0000 C CNN
@@
 $EndComp
 $Comp
-L GND #PWR06
+L GND #PWR5
 U 1 1 5426FD16
 P 2550 4850
-F 0 "#PWR06" H 2550 4850 30  0001 C CNN
+F 0 "#PWR5" H 2550 4850 30  0001 C CNN
 F 1 "GND" H 2550 4780 30  0001 C CNN
 F 2 "" H 2550 4850 60  0000 C CNN
@@
 L R R1
 U 1 1 5427C5CB
-P 4350 2750
-F 0 "R1" V 4430 2750 40  0000 C CNN
-F 1 "10k" V 4357 2751 40  0000 C CNN
-F 2 "~" V 4280 2750 30  0000 C CNN
-F 3 "~" H 4350 2750 30  0000 C CNN
-	1    4350 2750
-	1    0    0    -1
-$EndComp
-Wire Wire Line
-	3800 3000 4350 3000
-Text Label 4350 2500 0    60   ~ 0
+P 4550 3450
+F 0 "R1" V 4630 3450 40  0000 C CNN
+F 1 "10k" V 4557 3451 40  0000 C CNN
+F 2 "~" V 4480 3450 30  0000 C CNN
+F 3 "~" H 4550 3450 30  0000 C CNN
+	1    4550 3450
+	1    0    0    -1
+$EndComp
+Wire Wire Line
+	3800 3000 4550 3700
+Text Label 4550 3200 0    60   ~ 0
 3V3
 Wire Wire Line
@@
 $EndComp
 $Comp
-L GND #PWR07
+L GND #PWR1
 U 1 1 5427C6AA
 P 1450 2300
-F 0 "#PWR07" H 1450 2300 30  0001 C CNN
+F 0 "#PWR1" H 1450 2300 30  0001 C CNN
 F 1 "GND" H 1450 2230 30  0001 C CNN
 F 2 "" H 1450 2300 60  0000 C CNN
@@
 AREF
 $Comp
-L GND #PWR08
+L GND #PWR2
 U 1 1 5427C74B
 P 1700 2600
-F 0 "#PWR08" H 1700 2600 30  0001 C CNN
+F 0 "#PWR2" H 1700 2600 30  0001 C CNN
 F 1 "GND" H 1700 2530 30  0001 C CNN
 F 2 "" H 1700 2600 60  0000 C CNN
@@
 	4200 2050 4250 2050
 $Comp
-L GND #PWR09
+L GND #PWR8
 U 1 1 5427C845
 P 4550 2200
-F 0 "#PWR09" H 4550 2200 30  0001 C CNN
+F 0 "#PWR8" H 4550 2200 30  0001 C CNN
 F 1 "GND" H 4550 2130 30  0001 C CNN
 F 2 "" H 4550 2200 60  0000 C CNN
@@
 	4550 2150 4450 2150
 $Comp
-L GND #PWR010
+L GND #PWR3
 U 1 1 5427C883
 P 1700 4000
-F 0 "#PWR010" H 1700 4000 30  0001 C CNN
+F 0 "#PWR3" H 1700 4000 30  0001 C CNN
 F 1 "GND" H 1700 3930 30  0001 C CNN
 F 2 "" H 1700 4000 60  0000 C CNN
@@
 D13/SCK
 $Comp
-L 3V3 #PWR011
+L 3V3 #PWR6
 U 1 1 5427CC5F
 P 3300 4450
-F 0 "#PWR011" H 3300 4550 40  0001 C CNN
+F 0 "#PWR6" H 3300 4550 40  0001 C CNN
 F 1 "3V3" H 3300 4575 40  0000 C CNN
 F 2 "" H 3300 4450 60  0000 C CNN
@@
 $EndComp
 $Comp
-L +5V #PWR012
+L +5V #PWR4
 U 1 1 5427CC6E
 P 1950 4350
-F 0 "#PWR012" H 1950 4440 20  0001 C CNN
+F 0 "#PWR4" H 1950 4440 20  0001 C CNN
 F 1 "+5V" H 1950 4440 30  0000 C CNN
 F 2 "" H 1950 4350 60  0000 C CNN
@@
 	1950 4350 1950 4450
 Connection ~ 1950 4450
-Text Label 4350 3000 0    60   ~ 0
+Text Label 4550 3700 0    60   ~ 0
 RESET
 $Comp
@@
 	5050 3150 5050 2650
 Connection ~ 5050 2650
+$Comp
+L R R2
+U 1 1 544E0695
+P 4250 2700
+F 0 "R2" V 4330 2700 40  0000 C CNN
+F 1 "100K" V 4257 2701 40  0000 C CNN
+F 2 "~" V 4180 2700 30  0000 C CNN
+F 3 "~" H 4250 2700 30  0000 C CNN
+	1    4250 2700
+	1    0    0    -1
+$EndComp
+$Comp
+L R R3
+U 1 1 544E06A4
+P 4400 2700
+F 0 "R3" V 4480 2700 40  0000 C CNN
+F 1 "100K" V 4407 2701 40  0000 C CNN
+F 2 "~" V 4330 2700 30  0000 C CNN
+F 3 "~" H 4400 2700 30  0000 C CNN
+	1    4400 2700
+	1    0    0    -1
+$EndComp
+Wire Wire Line
+	3800 2400 4050 2400
+Wire Wire Line
+	4050 2400 4050 2450
+Wire Wire Line
+	4050 2450 4400 2450
+Connection ~ 4250 2450
+$Comp
+L GND #PWR7
+U 1 1 544E074A
+P 4250 3000
+F 0 "#PWR7" H 4250 3000 30  0001 C CNN
+F 1 "GND" H 4250 2930 30  0001 C CNN
+F 2 "" H 4250 3000 60  0000 C CNN
+F 3 "" H 4250 3000 60  0000 C CNN
+	1    4250 3000
+	1    0    0    -1
+$EndComp
+Wire Wire Line
+	4250 3000 4250 2950
+Text Label 4400 2950 0    60   ~ 0
+5V
 $EndSCHEMATC

Commit message: Increase header hole & pad size Fix MCP1800 reversed pins 2 & 3 Fix FTDI reversed TX & RX Add MISO & SCK labels Remove silk screen around mounting holes Increase pad size for 0603's for hand soldering
Parts:
- U2: value MCP1702T-3302E/CB -> MCP1700
Changed lines of the file:
@@
 Sheet 1 1
 Title ""
-Date "27 oct 2014"
+Date "8 dec 2014"
 Rev ""
 Comp ""
@@
 $EndComp
 $Comp
-L MCP1700 U2
-U 1 1 54257EE0
-P 2550 4500
-F 0 "U2" H 2700 4304 60  0000 C CNN
-F 1 "MCP1702T-3302E/CB" H 2550 4700 60  0000 C CNN
-F 2 "~" H 2550 4500 60  0000 C CNN
-F 3 "~" H 2550 4500 60  0000 C CNN
-	1    2550 4500
-	1    0    0    -1
-$EndComp
-$Comp
 L RFM12 U1
 U 1 1 54257F70
@@
 Text Label 5150 1050 0    60   ~ 0
 RESET
+Text Label 5300 1750 2    60   ~ 0
+D0/RX
 Text Label 5300 1650 2    60   ~ 0
-D0/RX
-Text Label 5300 1750 2    60   ~ 0
 D1/TX
 Text Label 5300 1850 2    60   ~ 0
@@
 NoConn ~ 5300 1950
 $Comp
-L GND #PWR10
+L GND #PWR01
 U 1 1 5425AD89
 P 5300 2050
-F 0 "#PWR10" H 5300 2050 30  0001 C CNN
+F 0 "#PWR01" H 5300 2050 30  0001 C CNN
 F 1 "GND" H 5300 1980 30  0001 C CNN
 F 2 "" H 5300 2050 60  0000 C CNN
@@
 5V
 $Comp
-L GND #PWR9
+L GND #PWR02
 U 1 1 5425ADEE
 P 5000 2850
-F 0 "#PWR9" H 5000 2850 30  0001 C CNN
+F 0 "#PWR02" H 5000 2850 30  0001 C CNN
 F 1 "GND" H 5000 2780 30  0001 C CNN
 F 2 "" H 5000 2850 60  0000 C CNN
@@
 5V
 $Comp
-L GND #PWR13
+L GND #PWR03
 U 1 1 5426FA0B
 P 6950 5000
-F 0 "#PWR13" H 6950 5000 30  0001 C CNN
+F 0 "#PWR03" H 6950 5000 30  0001 C CNN
 F 1 "GND" H 6950 4930 30  0001 C CNN
 F 2 "" H 6950 5000 60  0000 C CNN
@@
 	6350 4900 6300 4900
 $Comp
-L GND #PWR11
+L GND #PWR04
 U 1 1 5426FB80
 P 5350 5250
-F 0 "#PWR11" H 5350 5250 30  0001 C CNN
+F 0 "#PWR04" H 5350 5250 30  0001 C CNN
 F 1 "GND" H 5350 5180 30  0001 C CNN
 F 2 "" H 5350 5250 60  0000 C CNN
@@
 $EndComp
 $Comp
-L GND #PWR12
+L GND #PWR05
 U 1 1 5426FBC0
 P 6000 4100
-F 0 "#PWR12" H 6000 4100 30  0001 C CNN
+F 0 "#PWR05" H 6000 4100 30  0001 C CNN
 F 1 "GND" H 6000 4030 30  0001 C CNN
 F 2 "" H 6000 4100 60  0000 C CNN
@@
 $EndComp
 $Comp
-L GND #PWR5
+L GND #PWR06
 U 1 1 5426FD16
 P 2550 4850
-F 0 "#PWR5" H 2550 4850 30  0001 C CNN
+F 0 "#PWR06" H 2550 4850 30  0001 C CNN
 F 1 "GND" H 2550 4780 30  0001 C CNN
 F 2 "" H 2550 4850 60  0000 C CNN
@@
 $EndComp
 $Comp
-L GND #PWR1
+L GND #PWR07
 U 1 1 5427C6AA
 P 1450 2300
-F 0 "#PWR1" H 1450 2300 30  0001 C CNN
+F 0 "#PWR07" H 1450 2300 30  0001 C CNN
 F 1 "GND" H 1450 2230 30  0001 C CNN
 F 2 "" H 1450 2300 60  0000 C CNN
@@
 AREF
 $Comp
-L GND #PWR2
+L GND #PWR08
 U 1 1 5427C74B
 P 1700 2600
-F 0 "#PWR2" H 1700 2600 30  0001 C CNN
+F 0 "#PWR08" H 1700 2600 30  0001 C CNN
 F 1 "GND" H 1700 2530 30  0001 C CNN
 F 2 "" H 1700 2600 60  0000 C CNN
@@
 	4200 2050 4250 2050
 $Comp
-L GND #PWR8
+L GND #PWR09
 U 1 1 5427C845
 P 4550 2200
-F 0 "#PWR8" H 4550 2200 30  0001 C CNN
+F 0 "#PWR09" H 4550 2200 30  0001 C CNN
 F 1 "GND" H 4550 2130 30  0001 C CNN
 F 2 "" H 4550 2200 60  0000 C CNN
@@
 	4550 2150 4450 2150
 $Comp
-L GND #PWR3
+L GND #PWR010
 U 1 1 5427C883
 P 1700 4000
-F 0 "#PWR3" H 1700 4000 30  0001 C CNN
+F 0 "#PWR010" H 1700 4000 30  0001 C CNN
 F 1 "GND" H 1700 3930 30  0001 C CNN
 F 2 "" H 1700 4000 60  0000 C CNN
@@
 D13/SCK
 $Comp
-L 3V3 #PWR6
+L 3V3 #PWR011
 U 1 1 5427CC5F
 P 3300 4450
-F 0 "#PWR6" H 3300 4550 40  0001 C CNN
+F 0 "#PWR011" H 3300 4550 40  0001 C CNN
 F 1 "3V3" H 3300 4575 40  0000 C CNN
 F 2 "" H 3300 4450 60  0000 C CNN
@@
 $EndComp
 $Comp
-L +5V #PWR4
+L +5V #PWR012
 U 1 1 5427CC6E
 P 1950 4350
-F 0 "#PWR4" H 1950 4440 20  0001 C CNN
+F 0 "#PWR012" H 1950 4440 20  0001 C CNN
 F 1 "+5V" H 1950 4440 30  0000 C CNN
 F 2 "" H 1950 4350 60  0000 C CNN
@@
 Connection ~ 4250 2450
 $Comp
-L GND #PWR7
+L GND #PWR013
 U 1 1 544E074A
 P 4250 3000
-F 0 "#PWR7" H 4250 3000 30  0001 C CNN
+F 0 "#PWR013" H 4250 3000 30  0001 C CNN
 F 1 "GND" H 4250 2930 30  0001 C CNN
 F 2 "" H 4250 3000 60  0000 C CNN
@@
 Text Label 4400 2950 0    60   ~ 0
 5V
+$Comp
+L MCP1700 U2
+U 1 1 54855A58
+P 2550 4500
+F 0 "U2" H 2700 4304 60  0000 C CNN
+F 1 "MCP1700" H 2550 4700 60  0000 C CNN
+F 2 "~" H 2550 4500 60  0000 C CNN
+F 3 "~" H 2550 4500 60  0000 C CNN
+	1    2550 4500
+	1    0    0    -1
+$EndComp
 $EndSCHEMATC

Commit message: change to CP2104
Parts:
- added JP10: PWR_USB, S_JUMPER_2, symbol CONN_2
- JP6: value FTDI -> CP2104
Connections:
- wire segments 49 -> 67
- no-connect marks 5 -> 4
Other:
- moved on the sheet: C4
Changed lines of the file:
@@
 LIBS:rfm12
 LIBS:tiny328-cache
-EELAYER 27 0
+EELAYER 25 0
 EELAYER END
 $Descr A4 11693 8268
@@
 P 5650 1800
 F 0 "JP6" V 5600 1800 60  0000 C CNN
-F 1 "FTDI" V 5700 1800 60  0000 C CNN
+F 1 "CP2104" V 5700 1800 60  0000 C CNN
 F 2 "~" H 5650 1800 60  0000 C CNN
 F 3 "~" H 5650 1800 60  0000 C CNN
@@
 	1    0    0    -1
 $EndComp
-Text Label 5150 1050 0    60   ~ 0
+Text Label 5300 1050 0    60   ~ 0
 RESET
+Text Label 5300 1850 2    60   ~ 0
+D0/RX
+Text Label 5300 1950 2    60   ~ 0
+D1/TX
 Text Label 5300 1750 2    60   ~ 0
-D0/RX
-Text Label 5300 1650 2    60   ~ 0
-D1/TX
-Text Label 5300 1850 2    60   ~ 0
 5V
-NoConn ~ 5300 1950
-$Comp
-L GND #PWR01
+$Comp
+L GND #PWR10
 U 1 1 5425AD89
 P 5300 2050
-F 0 "#PWR01" H 5300 2050 30  0001 C CNN
+F 0 "#PWR10" H 5300 2050 30  0001 C CNN
 F 1 "GND" H 5300 1980 30  0001 C CNN
 F 2 "" H 5300 2050 60  0000 C CNN
@@
 L C C4
 U 1 1 5425AD9F
-P 5150 1250
-F 0 "C4" H 5150 1350 40  0000 L CNN
-F 1 "0.1uF" H 5156 1165 40  0000 L CNN
-F 2 "~" H 5188 1100 30  0000 C CNN
-F 3 "~" H 5150 1250 60  0000 C CNN
-	1    5150 1250
-	1    0    0    -1
-$EndComp
-Wire Wire Line
-	5150 1450 5150 1550
-Wire Wire Line
-	5150 1550 5300 1550
+P 5300 1250
+F 0 "C4" H 5300 1350 40  0000 L CNN
+F 1 "0.1uF" H 5306 1165 40  0000 L CNN
+F 2 "~" H 5338 1100 30  0000 C CNN
+F 3 "~" H 5300 1250 60  0000 C CNN
+	1    5300 1250
+	1    0    0    -1
+$EndComp
 Text Label 5300 2550 2    60   ~ 0
 5V
 $Comp
-L GND #PWR02
+L GND #PWR9
 U 1 1 5425ADEE
 P 5000 2850
-F 0 "#PWR02" H 5000 2850 30  0001 C CNN
+F 0 "#PWR9" H 5000 2850 30  0001 C CNN
 F 1 "GND" H 5000 2780 30  0001 C CNN
 F 2 "" H 5000 2850 60  0000 C CNN
@@
 5V
 $Comp
-L GND #PWR03
+L GND #PWR13
 U 1 1 5426FA0B
 P 6950 5000
-F 0 "#PWR03" H 6950 5000 30  0001 C CNN
+F 0 "#PWR13" H 6950 5000 30  0001 C CNN
 F 1 "GND" H 6950 4930 30  0001 C CNN
 F 2 "" H 6950 5000 60  0000 C CNN
@@
 	6350 4900 6300 4900
 $Comp
-L GND #PWR04
+L GND #PWR11
 U 1 1 5426FB80
 P 5350 5250
-F 0 "#PWR04" H 5350 5250 30  0001 C CNN
+F 0 "#PWR11" H 5350 5250 30  0001 C CNN
 F 1 "GND" H 5350 5180 30  0001 C CNN
 F 2 "" H 5350 5250 60  0000 C CNN
@@
 $EndComp
 $Comp
-L GND #PWR05
+L GND #PWR12
 U 1 1 5426FBC0
 P 6000 4100
-F 0 "#PWR05" H 6000 4100 30  0001 C CNN
+F 0 "#PWR12" H 6000 4100 30  0001 C CNN
 F 1 "GND" H 6000 4030 30  0001 C CNN
 F 2 "" H 6000 4100 60  0000 C CNN
@@
 $EndComp
 Wire Wire Line
-	6000 4100 6000 4000
-Wire Wire Line
-	6000 4000 5900 4000
-Wire Wire Line
-	5500 4000 5350 4000
+	6000 4000 6000 4100
+Wire Wire Line
+	5850 4000 6000 4000
+Wire Wire Line
+	5350 4000 5550 4000
 Wire Wire Line
 	5350 3900 5350 4200
@@
 $EndComp
 $Comp
-L GND #PWR06
+L GND #PWR5
 U 1 1 5426FD16
 P 2550 4850
-F 0 "#PWR06" H 2550 4850 30  0001 C CNN
+F 0 "#PWR5" H 2550 4850 30  0001 C CNN
 F 1 "GND" H 2550 4780 30  0001 C CNN
 F 2 "" H 2550 4850 60  0000 C CNN
@@
 	2550 4850 2550 4750
 Connection ~ 2550 4850
-Wire Wire Line
-	2950 4450 3450 4450
 $Comp
 L C C6
@@
 	1    0    0    -1
 $EndComp
-Wire Wire Line
-	3800 3000 4550 3700
 Text Label 4550 3200 0    60   ~ 0
 3V3
@@
 $EndComp
 $Comp
-L GND #PWR07
+L GND #PWR1
 U 1 1 5427C6AA
 P 1450 2300
-F 0 "#PWR07" H 1450 2300 30  0001 C CNN
+F 0 "#PWR1" H 1450 2300 30  0001 C CNN
 F 1 "GND" H 1450 2230 30  0001 C CNN
 F 2 "" H 1450 2300 60  0000 C CNN
@@
 $EndComp
 Wire Wire Line
-	1450 2250 1450 2300
+	1450 2200 1450 2300
 Connection ~ 1750 1850
 $Comp
@@
 AREF
 $Comp
-L GND #PWR08
+L GND #PWR2
 U 1 1 5427C74B
 P 1700 2600
-F 0 "#PWR08" H 1700 2600 30  0001 C CNN
+F 0 "#PWR2" H 1700 2600 30  0001 C CNN
 F 1 "GND" H 1700 2530 30  0001 C CNN
 F 2 "" H 1700 2600 60  0000 C CNN
@@
 $EndComp
 Wire Wire Line
-	1700 2600 1700 2550
+	1700 2500 1700 2600
 $Comp
 L CRYSTAL_SMD Y1
@@
 	4200 2050 4250 2050
 $Comp
-L GND #PWR09
+L GND #PWR8
 U 1 1 5427C845
 P 4550 2200
-F 0 "#PWR09" H 4550 2200 30  0001 C CNN
+F 0 "#PWR8" H 4550 2200 30  0001 C CNN
 F 1 "GND" H 4550 2130 30  0001 C CNN
 F 2 "" H 4550 2200 60  0000 C CNN
@@
 	4550 2150 4450 2150
 $Comp
-L GND #PWR010
+L GND #PWR3
 U 1 1 5427C883
 P 1700 4000
-F 0 "#PWR010" H 1700 4000 30  0001 C CNN
+F 0 "#PWR3" H 1700 4000 30  0001 C CNN
 F 1 "GND" H 1700 3930 30  0001 C CNN
 F 2 "" H 1700 4000 60  0000 C CNN
@@
 D13/SCK
 $Comp
-L 3V3 #PWR011
+L 3V3 #PWR6
 U 1 1 5427CC5F
-P 3300 4450
-F 0 "#PWR011" H 3300 4550 40  0001 C CNN
-F 1 "3V3" H 3300 4575 40  0000 C CNN
-F 2 "" H 3300 4450 60  0000 C CNN
-F 3 "" H 3300 4450 60  0000 C CNN
-	1    3300 4450
-	1    0    0    -1
-$EndComp
-$Comp
-L +5V #PWR012
+P 3200 4350
+F 0 "#PWR6" H 3200 4450 40  0001 C CNN
+F 1 "3V3" H 3200 4475 40  0000 C CNN
+F 2 "" H 3200 4350 60  0000 C CNN
+F 3 "" H 3200 4350 60  0000 C CNN
+	1    3200 4350
+	1    0    0    -1
+$EndComp
+$Comp
+L +5V #PWR4
 U 1 1 5427CC6E
 P 1950 4350
-F 0 "#PWR012" H 1950 4440 20  0001 C CNN
+F 0 "#PWR4" H 1950 4440 20  0001 C CNN
 F 1 "+5V" H 1950 4440 30  0000 C CNN
 F 2 "" H 1950 4350 60  0000 C CNN
@@
 Connection ~ 4250 2450
 $Comp
-L GND #PWR013
+L GND #PWR7
 U 1 1 544E074A
 P 4250 3000
-F 0 "#PWR013" H 4250 3000 30  0001 C CNN
+F 0 "#PWR7" H 4250 3000 30  0001 C CNN
 F 1 "GND" H 4250 2930 30  0001 C CNN
 F 2 "" H 4250 3000 60  0000 C CNN
@@
 $EndComp
 Wire Wire Line
-	4250 3000 4250 2950
+	4250 2850 4250 3000
 Text Label 4400 2950 0    60   ~ 0
 5V
@@
 	1    0    0    -1
 $EndComp
+$Comp
+L CONN_2 JP10
+U 1 1 554CCB84
+P 4650 1550
+F 0 "JP10" V 4600 1550 50  0000 C CNN
+F 1 "PWR_USB" V 4700 1550 40  0000 C CNN
+F 2 "S_JUMPER_2" H 4650 1550 60  0000 C CNN
+F 3 "~" H 4650 1550 60  0000 C CNN
+	1    4650 1550
+	-1   0    0    1
+$EndComp
+Wire Wire Line
+	5300 1100 5300 1050
+Wire Wire Line
+	5300 1650 5000 1650
+Text Label 5000 1350 2    60   ~ 0
+3V3
+Wire Wire Line
+	5000 1350 5000 1450
+Wire Wire Line
+	5300 1550 5300 1400
+Wire Wire Line
+	3300 4850 3300 4800
+Wire Wire Line
+	3050 4800 3050 4850
+Wire Wire Line
+	3050 4500 3050 4450
+Wire Wire Line
+	2950 4450 3450 4450
+Wire Wire Line
+	3300 4450 3300 4500
+Wire Wire Line
+	3200 4350 3200 4450
+Connection ~ 3200 4450
+Wire Wire Line
+	2050 4850 2050 4800
+Wire Wire Line
+	2050 4500 2050 4450
+Wire Wire Line
+	1700 2200 1700 2150
+Wire Wire Line
+	1450 1900 1450 1850
+Wire Wire Line
+	4250 2450 4250 2550
+Wire Wire Line
+	4400 2450 4400 2550
+Wire Wire Line
+	4400 2850 4400 2950
+Wire Wire Line
+	4550 3200 4550 3300
+Wire Wire Line
+	4550 3600 4150 3600
+Wire Wire Line
+	4150 3600 4150 3000
+Wire Wire Line
+	4150 3000 3800 3000
+Wire Wire Line
+	4550 3600 4550 3700
 $EndSCHEMATC
